File: esp-adap.brd (EAGLE design)
At the start: 27.9 x 14.9 mm, 3 parts

Commit message: board done
Parts:
- moved C1 1.27 mm to (14.0, 8.89)
- flipped JP1 to the bottom
Routing:
- net VCC: track 21.0 -> 0.00 mm
- net TXD: track 14.0 -> 28.1 mm
- net RXD: track 21.2 -> 10.5 mm
- net GND: track 8.70 -> 15.1 mm
- net CH_PD: track 9.92 -> 7.93 mm
- net RESET: track 8.01 -> 6.91 mm
- net GPIO2: track 5.39 -> 4.33 mm
- added copper zone on layer 1, net VCC
Other:
- board size 27.9 x 14.9 mm -> 26.7 x 12.4 mm
- board text added: "CH_PD"
- board text added: "GND"
- board text added: "GPIO0"
- board text added: "GPIO2"
- board text added: "RESET"
- board text added: "RXD"
- board text added: "TXD"
- board text added: "VCC"
- board text added: "github.com/fu0x11/esp8266-breadboard-adapter"

Commit message: updated board
Parts:
- JP2: device pinhead:1X10/90 -> pinhead:1X10
- moved JP2 3.81 mm to (12.7, 3.81)
Routing:
- net VCC: track 0.00 -> 11.6 mm
- net TXD: track 28.1 -> 22.8 mm
Other:
- board size 26.7 x 12.4 mm -> 26.5 x 11.2 mm
Changed lines of the file:
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@@
 <setting verticaltext="up"/>
 </settings>
-<grid distance="10" unitdist="mil" unit="mil" style="dots" multiple="1" display="yes" altdistance="0.025" altunitdist="inch" altunit="inch"/>
+<grid distance="5" unitdist="mil" unit="mil" style="dots" multiple="1" display="yes" altdistance="0.025" altunitdist="inch" altunit="inch"/>
 <layers>
 <layer number="1" name="Top" color="4" fill="1" visible="yes" active="yes"/>
@@
 <layer number="43" name="vRestrict" color="2" fill="10" visible="yes" active="yes"/>
 <layer number="44" name="Drills" color="7" fill="1" visible="no" active="yes"/>
-<layer number="45" name="Holes" color="7" fill="1" visible="no" active="yes"/>
+<layer number="45" name="Holes" color="7" fill="1" visible="yes" active="yes"/>
 <layer number="46" name="Milling" color="3" fill="1" visible="no" active="yes"/>
 <layer number="47" name="Measures" color="7" fill="1" visible="no" active="yes"/>
@@
 <board>
 <plain>
-<wire x1="-0.635" y1="0.635" x2="26.015" y2="0.635" width="0" layer="20"/>
-<wire x1="26.015" y1="0.635" x2="26.035" y2="6.985" width="0" layer="20"/>
-<wire x1="26.035" y1="6.985" x2="16.51" y2="6.985" width="0" layer="20"/>
-<wire x1="16.51" y1="6.985" x2="16.51" y2="13.005" width="0" layer="20"/>
-<wire x1="16.51" y1="13.005" x2="-0.635" y2="13.005" width="0" layer="20"/>
-<wire x1="-0.635" y1="13.005" x2="-0.635" y2="0.635" width="0" layer="20"/>
-<text x="25.146" y="6.096" size="0.4064" layer="26" rot="MR0">github.com/fu0x11/esp8266-breadboard-adapter</text>
+<wire x1="-0.635" y1="1.651" x2="25.888" y2="1.651" width="0" layer="20"/>
+<wire x1="25.888" y1="1.651" x2="25.908" y2="6.985" width="0" layer="20"/>
+<wire x1="25.908" y1="6.985" x2="16.51" y2="6.985" width="0" layer="20"/>
+<wire x1="16.51" y1="6.985" x2="16.51" y2="12.878" width="0" layer="20"/>
+<wire x1="16.51" y1="12.878" x2="-0.635" y2="12.878" width="0" layer="20"/>
+<wire x1="-0.635" y1="12.878" x2="-0.635" y2="1.651" width="0" layer="20"/>
+<text x="25.527" y="5.969" size="0.3556" layer="26" rot="MR0">github.com/fu0x11/esp8266-breadboard-adapter</text>
 <text x="0.254" y="5.588" size="0.4064" layer="25">CH_PD</text>
 <text x="3.048" y="5.588" size="0.4064" layer="25">GPIO2</text>
@@
 <text x="18.542" y="5.588" size="0.4064" layer="25">RXD</text>
 <text x="21.082" y="5.588" size="0.4064" layer="25">TXD</text>
+<hole x="0.381" y="11.938" drill="1"/>
 </plain>
 <attributes>
@@
 <param name="RoutingGrid" value="50mil"/>
 <param name="AutoGrid" value="1"/>
-<param name="Efforts" value="0"/>
+<param name="Efforts" value="2"/>
 <param name="TopRouterVariant" value="1"/>
 <param name="tpViaShape" value="round"/>
@@
 <element name="C1" library="resistor" package="C1206K" value="100u" x="13.97" y="8.89" rot="R270"/>
 <element name="JP1" library="pinhead" package="2X04" value="" x="6.35" y="8.89" rot="MR0"/>
-<element name="JP2" library="pinhead" package="1X10/90" value="" x="12.7" y="0" rot="R180"/>
+<element name="JP2" library="pinhead" package="1X10" value="" x="12.7" y="3.81" rot="R180"/>
 </elements>
 <signals>
@@
 <contactref element="JP1" pad="8"/>
 <contactref element="JP2" pad="2"/>
-<wire x1="19.6596" y1="1.8288" x2="21.4884" y2="3.6576" width="0.254" layer="16"/>
-<wire x1="5.9436" y1="1.8288" x2="19.6596" y2="1.8288" width="0.254" layer="16"/>
-<wire x1="5.0292" y1="2.7432" x2="5.9436" y2="1.8288" width="0.254" layer="16"/>
-<wire x1="5.0292" y1="5.0292" x2="5.0292" y2="2.7432" width="0.254" layer="16"/>
-<wire x1="3.6576" y1="6.4008" x2="5.0292" y2="5.0292" width="0.254" layer="16"/>
-<wire x1="2.0574" y1="6.4008" x2="3.6576" y2="6.4008" width="0.254" layer="16"/>
-<wire x1="1.3716" y1="7.0866" x2="2.0574" y2="6.4008" width="0.254" layer="16"/>
-<wire x1="1.3716" y1="8.9154" x2="1.3716" y2="7.0866" width="0.254" layer="16"/>
-<wire x1="2.5146" y1="10.0584" x2="1.3716" y2="8.9154" width="0.254" layer="16"/>
-<wire x1="21.4884" y1="3.6576" x2="21.59" y2="3.81" width="0.254" layer="16"/>
-<wire x1="2.5146" y1="10.0584" x2="2.54" y2="10.16" width="0.254" layer="16"/>
+<wire x1="2.54" y1="10.16" x2="3.048" y2="10.16" width="0.3048" layer="16"/>
+<wire x1="3.048" y1="10.16" x2="4.318" y2="8.89" width="0.3048" layer="16"/>
+<wire x1="4.318" y1="8.89" x2="14.732" y2="8.89" width="0.3048" layer="16"/>
+<wire x1="14.732" y1="8.89" x2="15.24" y2="8.382" width="0.3048" layer="16"/>
+<wire x1="15.24" y1="8.382" x2="15.24" y2="7.112" width="0.3048" layer="16"/>
+<wire x1="15.24" y1="7.112" x2="16.002" y2="6.35" width="0.3048" layer="16"/>
+<wire x1="16.002" y1="6.35" x2="19.558" y2="6.35" width="0.3048" layer="16"/>
+<wire x1="19.558" y1="6.35" x2="20.32" y2="5.588" width="0.3048" layer="16"/>
+<wire x1="20.32" y1="5.588" x2="20.32" y2="4.953" width="0.3048" layer="16"/>
+<wire x1="20.32" y1="4.953" x2="21.59" y2="3.81" width="0.3048" layer="16"/>
 </signal>
 <signal name="VCC">
@@
 <contactref element="JP1" pad="2"/>
 <contactref element="JP2" pad="4"/>
+<wire x1="10.287" y1="10.287" x2="13.9446" y2="10.287" width="0.254" layer="1"/>
+<wire x1="13.9446" y1="10.287" x2="13.97" y2="10.39" width="0.254" layer="1"/>
+<wire x1="10.287" y1="10.287" x2="10.16" y2="10.16" width="0.254" layer="1"/>
+<wire x1="16.4592" y1="5.2578" x2="16.4592" y2="3.8862" width="0.254" layer="1"/>
+<wire x1="15.3162" y1="6.4008" x2="16.4592" y2="5.2578" width="0.254" layer="1"/>
+<wire x1="15.3162" y1="8.4582" x2="15.3162" y2="6.4008" width="0.254" layer="1"/>
+<wire x1="14.1732" y1="9.6012" x2="15.3162" y2="8.4582" width="0.254" layer="1"/>
+<wire x1="14.1732" y1="10.287" x2="14.1732" y2="9.6012" width="0.254" layer="1"/>
+<wire x1="16.4592" y1="3.8862" x2="16.51" y2="3.81" width="0.254" layer="1"/>
+<wire x1="14.1732" y1="10.287" x2="13.97" y2="10.39" width="0.254" layer="1"/>
 <polygon width="0.4064" layer="1">
-<vertex x="-0.254" y="12.7"/>
-<vertex x="16.256" y="12.7"/>
+<vertex x="-0.254" y="12.573"/>
+<vertex x="16.256" y="12.573"/>
 <vertex x="16.256" y="6.604"/>
-<vertex x="25.654" y="6.604"/>
-<vertex x="25.654" y="1.016"/>
-<vertex x="-0.254" y="1.016"/>
+<vertex x="19.304" y="6.604"/>
+<vertex x="19.304" y="1.905"/>
+<vertex x="-0.254" y="1.905"/>
 </polygon>
 </signal>
